Commit message: floor urdf

File: data/robot_description/abb_linear_axis/urdf/abb_linear_axis_floor_two_robots.urdf (robot description, URDF)
Before this commit: robot linear_axis_two_robots, 22 links, 21 joints
Links:
- link axis: geometry collision mesh filename=package://abb_linear_axis/meshes/collision/axis_floor.stl; visual mesh filename=package://abb_linear_axis/meshes/visual/axis_floor.stl
- link cartA: geometry collision mesh filename=package://abb_linear_axis/meshes/collision/cart_floor.stl; visual mesh filename=package://abb_linear_axis/meshes/visual/cart_floor.stl
- link cartB: geometry collision mesh filename=package://abb_linear_axis/meshes/collision/cart_floor.stl; visual mesh filename=package://abb_linear_axis/meshes/visual/cart_floor.stl
Joints:
- joint cartA_joint: origin xyz=0.42 -0.02 3.104 rpy=3.14159265 0 0  -> xyz=0.42 -0.02 1.5 rpy=0 0 0 
- joint cartB_joint: origin xyz=16.08 -0.02 3.104 rpy=3.14159265 0 0  -> xyz=16.08 -0.02 1.5 rpy=0 0 0 
